File: powersupply_5v_v1.kicad_pcb (KiCad board)
At the start: 2 copper layers, 160.1 x 100 mm, 40 parts, among them P1 AC_INPUT, P2 POWER OUT, T1 TRANSFO2, U1 LM7805CT/NOPB, U2 LM7905CT/NOPB

Commit message: various pcb changes
Parts:
- moved REF** 154.6 mm to (143.6, 301.8)
- moved C6 19.7 mm to (175.6, 103.3), turned to 90 degrees
- moved C7 18.8 mm to (156.0, 104.1), turned to 90 degrees
- moved U1 7.88 mm to (168.2, 79.1), turned to 180 degrees
- moved C8 1.67 mm to (175.5, 122.7), turned to 90 degrees
- moved C5 1.56 mm to (156.3, 122.8), turned to 90 degrees
Routing:
- net (no net): track 0.00 -> 911.7 mm, vias 0 -> 2
- net GNDPWR: track 202.7 -> 0.00 mm, vias 1 -> 0
- net Net-(C13-Pad1): track 114.1 -> 67.9 mm
- net Net-(C14-Pad2): track 123.9 -> 78.4 mm, vias 1 -> 0
- net /NETURAL: track 32.0 -> 0.00 mm
- net /HOT: track 26.2 -> 0.00 mm
- net Net-(C1-Pad1): track 47.1 -> 23.1 mm
- net Net-(F1-Pad2): track 23.1 -> 0.00 mm
- net /V+: track 140.1 -> 119.7 mm
- net /REG_+5V: track 33.3 -> 15.5 mm
- net Net-(D8-Pad1): track 12.8 -> 0.00 mm
- net /V-: track 94.0 -> 105.7 mm
- net Net-(D7-Pad1): track 7.63 -> 0.00 mm
- net /REG_-5V: track 30.2 -> 31.5 mm
- net Net-(C3-Pad1): track 24.7 -> 23.7 mm
- added copper zone on B.Cu, net GNDPWR
- added copper zone on F.Cu, net GNDPWR

Commit message: added a small circuit for showing a LED indication when AC power is live
Parts:
- added G***: LOGO, logos:LOGO, B.Cu at (108.4, 137.5)
- added REF**: 3.5mmM3, mechanical:3.5mm_m3, F.Cu at (239.4, 156.9)
- added REF**: 3.5mmM3, mechanical:3.5mm_m3, F.Cu at (239.4, 62.9)
- added REF**: 3.5mmM3, mechanical:3.5mm_m3, F.Cu at (85.3, 62.8)
- added REF**: 3.5mmM3, mechanical:3.5mm_m3, F.Cu at (85.3, 157.0)
- added REF**: 3.5mmM3, mechanical:3.5mm_m3, F.Cu at (160.7, 62.9)
- added REF**: 3.5mmM3, mechanical:3.5mm_m3, F.Cu at (162.1, 157.0)
- added pad_2mm: VAL**, w_details:pad_2mm, B.Cu at (95.9, 111.5)
- added pad_2mm: VAL**, w_details:pad_2mm, B.Cu at (169.5, 143.8)
- added pad_2mm: VAL**, w_details:pad_2mm, B.Cu at (172.9, 143.8)
- added pad_2mm: VAL**, w_details:pad_2mm, B.Cu at (95.8, 117.0)
- added pad_2mm: VAL**, w_details:pad_2mm, B.Cu at (95.9, 124.4)
- added pad_2mm: VAL**, w_details:pad_2mm, F.Cu at (231.2, 125.8)
- added pad_2mm: VAL**, w_details:pad_2mm, F.Cu at (230.7, 100.9)
- added pad_2mm: VAL**, w_details:pad_2mm, F.Cu at (170.6, 70.6)
- added pad_2mm: VAL**, w_details:pad_2mm, F.Cu at (167.8, 70.6)
- added pad_2mm: VAL**, w_details:pad_2mm, F.Cu at (165.0, 70.6)
- added pad_2mm: VAL**, w_details:pad_2mm, B.Cu at (166.1, 143.9)
- U1: value LM7805CT/NOPB -> LM7805CT
- U2: value LM7905CT/NOPB -> LM7905CT
Routing:
- net Net-(C14-Pad2): track 78.4 -> 126.2 mm, vias 0 -> 1
- net Net-(C13-Pad1): track 67.9 -> 115.6 mm
- net /NETURAL: track 0.00 -> 43.1 mm
- net GNDPWR: track 0.00 -> 41.4 mm
- net /V+: track 119.7 -> 152.6 mm
- net /HOT: track 0.00 -> 25.4 mm
- net Net-(C1-Pad1): track 23.1 -> 44.8 mm
- net Net-(F1-Pad2): track 0.00 -> 16.8 mm
- net /REG_+5V: track 15.5 -> 29.3 mm
- net Net-(D8-Pad1): track 0.00 -> 12.6 mm
- net Net-(D7-Pad1): track 0.00 -> 8.05 mm
Other:
- board text added: "+"
- board text added: "+5"
- board text added: "-5"
- board text added: "AC INPUT"
- board text added: "EARTH"
- board text added: "GND"
- board text added: "HOT"
- board text added: "Hornosty.com"
- board text added: "NETURAL"
- board text added: "OUT"
- board text added: "V+"
- board text added: "V-"
